File: kicad_board/multieff.kicad_pcb (KiCad board)
At the start: 2 copper layers, 120 x 80 mm, 45 parts, among them J1 Wha1, U1 MCP23017_SO, U2 MCP23017_SO, U4 ADS1115IDGS

Commit message: Update project name
Other:
- board text added: "https://github.com/kleag/riffpi"
- board text removed: "https://github.com/kleag/kleagmfx"
Changed lines of the file:
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@@
 		)
 	)
-	(gr_text "https://github.com/kleag/kleagmfx"
+	(gr_text "https://github.com/kleag/riffpi"
 		(at 122.5 58.5 0)
 		(layer "Dwgs.User")
